Commit message: Further improvements to the computational efficiency of the sim. For the example polytunnel/actor configurations in this package the real-time factor should now be 0.97. Collision properties of the type-2 actor have been adjusted.

File: rasberry_gazebo/urdf/actor_model.xacro (robot description, xacro)
@@ -3,5 +3,5 @@
   <link name="u_base_link">
     <inertial>
-      <pose>0 -0.1 0.05 0 0 0</pose>
+      <pose>0 -0.1 0.95 0 0 0</pose>
       <mass value="80.0"/>
       <inertia
@@ -18,4 +18,10 @@
       <geometry>
         <box size="0.5 0.35 0.02"/>
+      </geometry>
+    </collision>
+    <collision name="person">
+      <origin xyz="0 0 0.02" rpy="0.04 0 0"/>
+      <geometry>
+        <mesh filename="model://person_standing/meshes/standing.dae"/>
       </geometry>
     </collision>
