Commit message: The type 2 actor's laser scanner is now included in the tf tree. The launch file 'thorvald_world_AB.launch' now launches the Thorvald robot model into the gazebo world. The README.md has been adjusted to reflect these changes.

File: rasberry_gazebo/urdf/actor_laser.xacro (robot description, xacro)
@@ -2,7 +2,7 @@
 <robot name="laser" xmlns:xacro="http://www.ros.org/wiki/xacro">
   <!-- hokuyo -->
-  <gazebo reference="$(arg tf_prefix)/base_footprint">
+  <gazebo reference="$(arg tf_prefix)/hokuyo">
     <sensor type="ray" name="head_hokuyo_sensor">
-      <pose>0 0 1 0 0 0</pose>
+      <pose>0 0 0 0 0 0</pose>
       <visualize>false</visualize>
       <update_rate>40</update_rate>

File: rasberry_gazebo/urdf/actor_model.xacro (robot description, xacro)
@@ -34,4 +34,11 @@
   </link>
   <link name="$(arg tf_prefix)/base_footprint"/>
+  <link name="$(arg tf_prefix)/hokuyo"/>
+  <joint name="base_link_to_hokuyo" type="fixed">
+    <parent link="$(arg tf_prefix)/base_link"/>
+    <child link="$(arg tf_prefix)/hokuyo"/>
+    <axis xyz="0 1 0" />
+    <origin xyz="0 0 1" rpy="0 0 0"/>
+  </joint>
   <!-- For odometry -->
   <joint name="$(arg tf_prefix)/base_footprint_fixed" type="fixed">
