Commit message: Fixed the type-2 actor's tf trees. Thank you Gautham P Das!

File: rasberry_gazebo/urdf/actor.xacro (robot description, xacro)
@@ -3,12 +3,3 @@
   <xacro:include filename="$(find rasberry_gazebo)/urdf/actor_model.xacro"/>
   <xacro:include filename="$(find rasberry_gazebo)/urdf/actor_laser.xacro"/>
-  <gazebo>
-    <plugin name="object_controller" filename="libgazebo_ros_planar_move.so">
-      <commandTopic>cmd_vel</commandTopic>
-      <odometryTopic>u_odom</odometryTopic>
-      <odometryFrame>u_odom</odometryFrame>
-      <odometryRate>20.0</odometryRate>
-      <robotBaseFrame>u_base_footprint</robotBaseFrame>
-    </plugin>
-  </gazebo>
 </robot>

File: rasberry_gazebo/urdf/actor_laser.xacro (robot description, xacro)
@@ -2,5 +2,5 @@
 <robot name="laser" xmlns:xacro="http://www.ros.org/wiki/xacro">
   <!-- hokuyo -->
-  <gazebo reference="u_base_footprint">
+  <gazebo reference="$(arg tf_prefix)/base_footprint">
     <sensor type="ray" name="head_hokuyo_sensor">
       <pose>0 0 1 0 0 0</pose>
@@ -29,5 +29,5 @@
       <plugin name="gazebo_ros_head_hokuyo_controller" filename="libgazebo_ros_laser.so">
         <topicName>scan</topicName>
-        <frameName>u_base_footprint</frameName>
+        <frameName>base_footprint</frameName>
       </plugin>
     </sensor>

File: rasberry_gazebo/urdf/actor_model.xacro (robot description, xacro)
@@ -1,5 +1,5 @@
 <?xml version="1.0"?>
 <robot name="actor" xmlns:xacro="http://www.ros.org/wiki/xacro">
-  <link name="u_base_link">
+  <link name="$(arg tf_prefix)/base_link">
     <inertial>
       <pose>0 -0.1 0.95 0 0 0</pose>
@@ -33,10 +33,22 @@
     </visual>
   </link>
-  <link name="u_base_footprint"/>
+  <link name="$(arg tf_prefix)/base_footprint"/>
   <!-- For odometry -->
-  <joint name="base_footprint_fixed" type="fixed">
+  <joint name="$(arg tf_prefix)/base_footprint_fixed" type="fixed">
     <origin xyz="0 0 0.09" rpy="0 0 0"/>
-    <parent link="u_base_footprint"/>
-    <child  link="u_base_link"/>
+    <parent link="$(arg tf_prefix)/base_footprint"/>
+    <child  link="$(arg tf_prefix)/base_link"/>
   </joint>
+  <gazebo reference="$(arg tf_prefix)/base_link">
+    <selfCollide>false</selfCollide>
+  </gazebo>
+  <gazebo>
+    <plugin name="object_controller" filename="libgazebo_ros_planar_move.so">
+      <commandTopic>cmd_vel</commandTopic>
+      <odometryTopic>odom</odometryTopic>
+      <odometryFrame>$(arg tf_prefix)/odom</odometryFrame>
+      <odometryRate>20.0</odometryRate>
+      <robotBaseFrame>$(arg tf_prefix)/base_footprint</robotBaseFrame>
+    </plugin>
+  </gazebo>
 </robot>

Commit message: Some changes for Jaime to check.

File: rasberry_gazebo/urdf/actor.xacro (robot description, xacro)
@@ -1,5 +1,107 @@
 <?xml version="1.0"?>
-<robot name="actor" xmlns:xacro="http://www.ros.org/wiki/xacro">
-  <xacro:include filename="$(find rasberry_gazebo)/urdf/actor_model.xacro"/>
-  <xacro:include filename="$(find rasberry_gazebo)/urdf/actor_laser.xacro"/>
+<robot xmlns:xacro="http://www.ros.org/wiki/xacro" name="actor">
+  <xacro:arg name="robot_name" default=""/>
+  <xacro:arg name="tf_prefix" default=""/>
+<!-- PLUGINS -->
+<gazebo>
+  <plugin name="object_controller" filename="libgazebo_ros_planar_move.so">
+    <alwaysOn>true</alwaysOn>
+    <updateRate>20</updateRate>
+    <robotNamespace>$(arg robot_name)</robotNamespace>
+    <commandTopic>cmd_vel</commandTopic>
+    <odometryTopic>odom</odometryTopic>
+    <odometryFrame>$(arg tf_prefix)/odom</odometryFrame>
+    <odometryRate>20</odometryRate>
+    <robotBaseFrame>$(arg tf_prefix)/base_footprint</robotBaseFrame>
+  </plugin>
+</gazebo>
+<!-- CREATE LINKS -->
+<link name="$(arg tf_prefix)/base_footprint"/>
+<link name="$(arg tf_prefix)/base_link">
+  <inertial>
+    <pose>0 -0.1 0.95 0 0 0</pose>
+    <mass value="80.0"/>
+    <inertia
+      ixx="0.2085"
+      ixy="0.2385"
+      ixz="0.2385"
+      iyy="0.2385"
+      iyz="0.2385"
+      izz="0.2949"
+            />
+  </inertial>
+  <collision name="box">
+    <origin xyz="0 -0.1 0.01" rpy="0 0 0"/>
+    <geometry>
+      <box size="0.5 0.35 0.02"/>
+    </geometry>
+  </collision>
+  <collision name="person">
+    <origin xyz="0 0 0.02" rpy="0.04 0 0"/>
+    <geometry>
+      <mesh filename="model://person_standing/meshes/standing.dae"/>
+    </geometry>
+  </collision>
+  <visual name="visual">
+    <origin xyz="0 0 0.02" rpy="0.04 0 1.54"/>
+    <geometry>
+      <mesh filename="model://person_standing/meshes/standing.dae"/>
+    </geometry>
+  </visual>
+</link>
+<gazebo reference="$(arg tf_prefix)/base_link">
+  <selfCollide>false</selfCollide>
+</gazebo>
+<link name="$(arg tf_prefix)/hokuyo"/>
+<!-- CREATE JOINTS -->
+<!-- For odometry -->
+<joint name="$(arg tf_prefix)/base_footprint_to_base_link" type="fixed">
+  <parent link="$(arg tf_prefix)/base_footprint"/>
+  <child  link="$(arg tf_prefix)/base_link"/>
+  <origin xyz="0 0 0.09" rpy="0 0 0"/>
+</joint>
+<joint name="$(arg tf_prefix)/base_link_to_hokuyo" type="fixed">
+  <parent link="$(arg tf_prefix)/base_link"/>
+  <child link="$(arg tf_prefix)/hokuyo"/>
+  <axis xyz="0 1 0" />
+  <origin xyz="0 0 1" rpy="0 0 0"/>
+</joint>
+<!-- CREATE SENSORS -->
+  <gazebo reference="$(arg tf_prefix)/hokuyo">
+      <sensor name="head_hokuyo_sensor" type="ray">
+      <pose>0.1 0 0 0 0 0</pose>
+      <visualize>true</visualize>
+      <update_rate>40</update_rate>
+      <always_on>1</always_on>
+      <ray>
+        <scan>
+          <horizontal>
+            <samples>720</samples>
+            <resolution>1</resolution>
+            <min_angle>-1.570796</min_angle>
+            <max_angle>1.570796</max_angle>
+          </horizontal>
+        </scan>
+        <range>
+          <min>0.5</min>
+          <max>30.0</max>
+          <resolution>0.01</resolution>
+        </range>
+        <noise>
+          <type>gaussian</type>
+          <!-- Noise parameters based on published spec for Hokuyo laser
+               achieving "+-30mm" accuracy at range < 10m.  A mean of 0.0m and
+               stddev of 0.01m will put 99.7% of samples within 0.03m of the true
+               reading. -->
+          <mean>0.0</mean>
+          <stddev>0.01</stddev>
+        </noise>
+      </ray>
+        <plugin name="hokuyo_node" filename="libgazebo_ros_laser.so">
+        <topicName>scan</topicName>
+        <!--frameName>$(arg tf_prefix)/hokuyo</frameName-->
+        <frameName>hokuyo</frameName>
+        </plugin>
+    </sensor>
+  </gazebo>
 </robot>

Commit message: More changes for testing ...

File: rasberry_gazebo/urdf/actor.xacro (robot description, xacro)
@@ -37,4 +37,10 @@
     </geometry>
   </collision>
+  <visual name="box">
+    <origin xyz="0 -0.1 0.01" rpy="0 0 0"/>
+    <geometry>
+      <box size="0.5 0.35 0.02"/>
+    </geometry>
+  </visual>
   <collision name="person">
     <origin xyz="0 0 0.02" rpy="0.04 0 0"/>

Commit message: The package rasberry_actors has been subsumed into rasberry_gazebo. Move base has been implemented for multiple actors using teb local planner. A node has been created for publishing sequences of nav goals - can be used for actors or robots (see rasberry_gazebo/scripts/move_base_seq.py). A launch file for use with the physical robot (no sim elements) only has been made. See rasberry_gazebo/launch/thorvald_realtime.launch.
To fix: actors only avoiding obstacles in the no go map. Probably laser data not making it into local costmap.

File: rasberry_gazebo/urdf/actor.xacro (robot description, xacro)
@@ -71,10 +71,10 @@
   <child link="$(arg tf_prefix)/hokuyo"/>
   <axis xyz="0 1 0" />
-  <origin xyz="0 0 1" rpy="0 0 0"/>
+  <origin xyz="0 0 0.6" rpy="0 0 0"/>
 </joint>
 <!-- CREATE SENSORS -->
 <gazebo reference="$(arg tf_prefix)/hokuyo">
-  <sensor name="$(arg actor_name)_hokuyo_sensor" type="ray">
-    <pose>0.1 0 0 0 0 0</pose>
+  <sensor name="$(arg actor_name)_hokuyo_sensor" type="gpu_ray">
+    <pose>0 0 0 0 0 0</pose>
     <visualize>true</visualize>
     <update_rate>40</update_rate>
@@ -100,5 +100,5 @@
       </noise>
     </ray>
-    <plugin name="$(arg actor_name)_hokuyo_node" filename="libgazebo_ros_laser.so">
+    <plugin name="$(arg actor_name)_hokuyo_node" filename="libgazebo_ros_gpu_laser.so">
       <topicName>scan</topicName>
       <frameName>hokuyo</frameName>

Commit message: Fixed error causing the robots laser scan data from getting into the actor's local costmap. (#102)
Some tuning of the teb local planner for the actors - actors now avoid each other and the robot and can navigate the rows smoothly.
Laser model samples have been reduced from 720 to 36 - no issues with performance.

File: rasberry_gazebo/urdf/actor.xacro (robot description, xacro)
@@ -3,106 +3,106 @@
   <xacro:arg name="actor_name" default=""/>
   <xacro:arg name="tf_prefix" default=""/>
-<!-- PLUGINS -->
-<gazebo>
-  <plugin name="$(arg actor_name)_object_controller" filename="libgazebo_ros_planar_move.so">
-    <alwaysOn>true</alwaysOn>
-    <updateRate>20</updateRate>
-    <robotNamespace>$(arg actor_name)</robotNamespace>
-    <commandTopic>cmd_vel</commandTopic>
-    <odometryTopic>odom</odometryTopic>
-    <odometryFrame>$(arg tf_prefix)/odom</odometryFrame>
-    <odometryRate>20</odometryRate>
-    <robotBaseFrame>$(arg tf_prefix)/base_footprint</robotBaseFrame>
-  </plugin>
-</gazebo>
-<!-- CREATE LINKS -->
-<link name="$(arg tf_prefix)/base_footprint"/>
-<link name="$(arg tf_prefix)/base_link">
-  <inertial>
-    <pose>0 -0.1 0.95 0 0 0</pose>
-    <mass value="80.0"/>
-    <inertia
-      ixx="0.2085"
-      ixy="0.2385"
-      ixz="0.2385"
-      iyy="0.2385"
-      iyz="0.2385"
-      izz="0.2949"
-            />
-  </inertial>
-  <collision name="$(arg actor_name)_box">
-    <origin xyz="0 0 0.01" rpy="0 0 0"/>
-    <geometry>
-      <box size="0.5 0.35 0.02"/>
-    </geometry>
-  </collision>
-  <!--visual name="box">
-    <origin xyz="0 0 0.05" rpy="0 0 0"/>
-    <geometry>
-      <box size="0.5 0.35 0.02"/>
-    </geometry>
-  </visual-->
-  <collision name="$(arg actor_name)_person">
-    <origin xyz="0 0 0.02" rpy="0.04 0 0"/>
-    <geometry>
-      <mesh filename="model://person_standing/meshes/standing.dae"/>
-    </geometry>
-  </collision>
-  <visual name="$(arg actor_name)_visual">
-    <origin xyz="0 0 0.02" rpy="0.04 0 1.54"/>
-    <geometry>
-      <mesh filename="model://person_standing/meshes/standing.dae"/>
-    </geometry>
-  </visual>
-</link>
-<gazebo reference="$(arg tf_prefix)/base_link">
-  <selfCollide>false</selfCollide>
-</gazebo>
-<link name="$(arg tf_prefix)/hokuyo"/>
-<!-- CREATE JOINTS -->
-<!-- For odometry -->
-<joint name="$(arg tf_prefix)/base_footprint_to_base_link" type="fixed">
-  <parent link="$(arg tf_prefix)/base_footprint"/>
-  <child  link="$(arg tf_prefix)/base_link"/>
-  <origin xyz="0 0 0.09" rpy="0 0 0"/>
-</joint>
-<joint name="$(arg tf_prefix)/base_link_to_hokuyo" type="fixed">
-  <parent link="$(arg tf_prefix)/base_link"/>
-  <child link="$(arg tf_prefix)/hokuyo"/>
-  <axis xyz="0 1 0" />
-  <origin xyz="0 0 0.6" rpy="0 0 0"/>
-</joint>
-<!-- CREATE SENSORS -->
-<gazebo reference="$(arg tf_prefix)/hokuyo">
-  <sensor name="$(arg actor_name)_hokuyo_sensor" type="gpu_ray">
-    <pose>0 0 0 0 0 0</pose>
-    <visualize>true</visualize>
-    <update_rate>40</update_rate>
-    <always_on>1</always_on>
-    <ray>
-      <scan>
-        <horizontal>
-          <samples>720</samples>
-          <resolution>1</resolution>
-          <min_angle>-1.570796</min_angle>
-          <max_angle>1.570796</max_angle>
-        </horizontal>
-      </scan>
-      <range>
-        <min>0.5</min>
-        <max>30.0</max>
-        <resolution>0.01</resolution>
-      </range>
-      <noise>
-        <type>gaussian</type>
-        <mean>0.0</mean>
-        <stddev>0.01</stddev>
-      </noise>
-    </ray>
-    <plugin name="$(arg actor_name)_hokuyo_node" filename="libgazebo_ros_gpu_laser.so">
-      <topicName>scan</topicName>
-      <frameName>hokuyo</frameName>
+  <!-- PLUGINS -->
+  <gazebo>
+    <plugin name="$(arg actor_name)_object_controller" filename="libgazebo_ros_planar_move.so">
+      <alwaysOn>true</alwaysOn>
+      <updateRate>20.0</updateRate>
+      <robotNamespace>$(arg actor_name)</robotNamespace>
+       <commandTopic>cmd_vel</commandTopic>
+      <odometryTopic>odom</odometryTopic>
+      <odometryFrame>$(arg tf_prefix)/odom</odometryFrame>
+      <odometryRate>20.0</odometryRate>
+      <robotBaseFrame>$(arg tf_prefix)/base_footprint</robotBaseFrame>
     </plugin>
-  </sensor>
-</gazebo>
+  </gazebo>
+  <!-- CREATE LINKS -->
+  <link name="$(arg tf_prefix)/base_footprint"/>
+  <link name="$(arg tf_prefix)/base_link">
+    <inertial>
+      <pose>0 0 0.95 0 0 0</pose>
+      <mass value="80.0"/>
+      <inertia
+        ixx="0.2085"
+        ixy="0.2385"
+        ixz="0.2385"
+        iyy="0.2385"
+        iyz="0.2385"
+        izz="0.2949"
+              />
+    </inertial>
+    <collision name="$(arg actor_name)_box">
+      <origin xyz="0 0 0.01" rpy="0 0 0"/>
+      <geometry>
+        <box size="0.5 0.35 0.02"/>
+      </geometry>
+    </collision>
+    <!--visual name="box">
+      <origin xyz="0 0 0.05" rpy="0 0 0"/>
+      <geometry>
+        <box size="0.5 0.35 0.02"/>
+      </geometry>
+    </visual-->
+    <collision name="$(arg actor_name)_person">
+      <origin xyz="0 0 0.02" rpy="0.04 0 0"/>
+      <geometry>
+        <mesh filename="model://person_standing/meshes/standing.dae"/>
+      </geometry>
+    </collision>
+    <visual name="$(arg actor_name)_visual">
+      <origin xyz="0 0 0.02" rpy="0.04 0 1.54"/>
+      <geometry>
+        <mesh filename="model://person_standing/meshes/standing.dae"/>
+      </geometry>
+    </visual>
+  </link>
+  <gazebo reference="$(arg tf_prefix)/base_link">
+    <selfCollide>false</selfCollide>
+  </gazebo>
+  <link name="$(arg tf_prefix)/hokuyo"/>
+  <!-- CREATE JOINTS -->
+  <!-- For odometry -->
+  <joint name="$(arg tf_prefix)/base_footprint_to_base_link" type="fixed">
+    <parent link="$(arg tf_prefix)/base_footprint"/>
+    <child  link="$(arg tf_prefix)/base_link"/>
+    <origin xyz="0 0 0.09" rpy="0 0 0"/>
+  </joint>
+  <joint name="$(arg tf_prefix)/base_link_to_hokuyo" type="fixed">
+    <parent link="$(arg tf_prefix)/base_link"/>
+    <child link="$(arg tf_prefix)/hokuyo"/>
+    <axis xyz="0 1 0" />
+    <origin xyz="0.175 0 0.73" rpy="0 0 0"/>
+  </joint>
+  <!-- CREATE SENSORS -->
+  <gazebo reference="$(arg tf_prefix)/hokuyo">
+    <sensor name="$(arg actor_name)_hokuyo_sensor" type="gpu_ray">
+      <pose>0 0 0 0 0 0</pose>
+      <visualize>false</visualize>
+      <update_rate>40</update_rate>
+      <always_on>1</always_on>
+      <ray>
+        <scan>
+          <horizontal>
+            <samples>36</samples>
+            <resolution>1</resolution>
+            <min_angle>-1.570796</min_angle>
+            <max_angle>1.570796</max_angle>
+          </horizontal>
+        </scan>
+        <range>
+          <min>0.1</min>
+          <max>50.0</max>
+          <resolution>0.01</resolution>
+        </range>
+        <!--noise>
+          <type>gaussian</type>
+          <mean>0.0</mean>
+          <stddev>0.01</stddev>
+        </noise-->
+      </ray>
+      <plugin name="$(arg actor_name)_hokuyo_node" filename="libgazebo_ros_gpu_laser.so">
+        <topicName>scan</topicName>
+        <frameName>hokuyo</frameName>
+      </plugin>
+    </sensor>
+  </gazebo>
 </robot>
