Commit message: Seperated the gazebo world with polytunnels and actor spawning into seperate packages (rasberry_gazebo and actor_gazebo, respectively). There is also a rasberry_bringup package that launches everything together

File: rasberry_actors/urdf/actor.xacro (robot description, xacro)
@@ -32,15 +32,15 @@
   </inertial>
   <collision name="box">
-    <origin xyz="0 -0.1 0.01" rpy="0 0 0"/>
+    <origin xyz="0 0 0.01" rpy="0 0 0"/>
     <geometry>
       <box size="0.5 0.35 0.02"/>
     </geometry>
   </collision>
-  <visual name="box">
-    <origin xyz="0 -0.1 0.01" rpy="0 0 0"/>
+  <!--visual name="box">
+    <origin xyz="0 0 0.05" rpy="0 0 0"/>
     <geometry>
       <box size="0.5 0.35 0.02"/>
     </geometry>
-  </visual>
+  </visual-->
   <collision name="person">
     <origin xyz="0 0 0.02" rpy="0.04 0 0"/>

Commit message: Changes for testing (not to be merged)

File: rasberry_actors/urdf/actor.xacro (robot description, xacro)
@@ -1,12 +1,12 @@
 <?xml version="1.0"?>
 <robot xmlns:xacro="http://www.ros.org/wiki/xacro" name="actor">
-  <xacro:arg name="robot_name" default=""/>
+  <xacro:arg name="actor_name" default=""/>
   <xacro:arg name="tf_prefix" default=""/>
 <!-- PLUGINS -->
 <gazebo>
-  <plugin name="object_controller" filename="libgazebo_ros_planar_move.so">
+  <plugin name="$(arg actor_name)_object_controller" filename="libgazebo_ros_planar_move.so">
     <alwaysOn>true</alwaysOn>
     <updateRate>20</updateRate>
-    <robotNamespace>$(arg robot_name)</robotNamespace>
+    <robotNamespace>$(arg actor_name)</robotNamespace>
     <commandTopic>cmd_vel</commandTopic>
     <odometryTopic>odom</odometryTopic>
@@ -31,5 +31,5 @@
             />
   </inertial>
-  <collision name="box">
+  <collision name="$(arg actor_name)_box">
     <origin xyz="0 0 0.01" rpy="0 0 0"/>
     <geometry>
@@ -43,5 +43,5 @@
     </geometry>
   </visual-->
-  <collision name="person">
+  <collision name="$(arg actor_name)_person">
     <origin xyz="0 0 0.02" rpy="0.04 0 0"/>
     <geometry>
@@ -49,5 +49,5 @@
     </geometry>
   </collision>
-  <visual name="visual">
+  <visual name="$(arg actor_name)_visual">
     <origin xyz="0 0 0.02" rpy="0.04 0 1.54"/>
     <geometry>
@@ -74,40 +74,35 @@
 </joint>
 <!-- CREATE SENSORS -->
-  <gazebo reference="$(arg tf_prefix)/hokuyo">
-      <sensor name="head_hokuyo_sensor" type="ray">
-      <pose>0.1 0 0 0 0 0</pose>
-      <visualize>true</visualize>
-      <update_rate>40</update_rate>
-      <always_on>1</always_on>
-      <ray>
-        <scan>
-          <horizontal>
-            <samples>720</samples>
-            <resolution>1</resolution>
-            <min_angle>-1.570796</min_angle>
-            <max_angle>1.570796</max_angle>
-          </horizontal>
-        </scan>
-        <range>
-          <min>0.5</min>
-          <max>30.0</max>
-          <resolution>0.01</resolution>
-        </range>
-        <noise>
-          <type>gaussian</type>
-          <!-- Noise parameters based on published spec for Hokuyo laser
-               achieving "+-30mm" accuracy at range < 10m.  A mean of 0.0m and
-               stddev of 0.01m will put 99.7% of samples within 0.03m of the true
-               reading. -->
-          <mean>0.0</mean>
-          <stddev>0.01</stddev>
-        </noise>
-      </ray>
-        <plugin name="hokuyo_node" filename="libgazebo_ros_laser.so">
-        <topicName>scan</topicName>
-        <!--frameName>$(arg tf_prefix)/hokuyo</frameName-->
-        <frameName>hokuyo</frameName>
-        </plugin>
-    </sensor>
-  </gazebo>
+<gazebo reference="$(arg tf_prefix)/hokuyo">
+  <sensor name="$(arg actor_name)_hokuyo_sensor" type="ray">
+    <pose>0.1 0 0 0 0 0</pose>
+    <visualize>true</visualize>
+    <update_rate>40</update_rate>
+    <always_on>1</always_on>
+    <ray>
+      <scan>
+        <horizontal>
+          <samples>720</samples>
+          <resolution>1</resolution>
+          <min_angle>-1.570796</min_angle>
+          <max_angle>1.570796</max_angle>
+        </horizontal>
+      </scan>
+      <range>
+        <min>0.5</min>
+        <max>30.0</max>
+        <resolution>0.01</resolution>
+      </range>
+      <noise>
+        <type>gaussian</type>
+        <mean>0.0</mean>
+        <stddev>0.01</stddev>
+      </noise>
+    </ray>
+    <plugin name="$(arg actor_name)_hokuyo_node" filename="libgazebo_ros_laser.so">
+      <topicName>scan</topicName>
+      <frameName>hokuyo</frameName>
+    </plugin>
+  </sensor>
+</gazebo>
 </robot>
