Commit message: New Config file and Velodyne Frame in xacro (#109)

File: rasberry_bringup/urdf/norway_robot_003_sensors.xacro (robot description, xacro)
@@ -6,4 +6,5 @@
   <link name="$(arg tf_prefix)/septentrio"/>
   <link name="$(arg tf_prefix)/xsens"/>
+  <link name="$(arg tf_prefix)/velodyne"/>
   <!-- Hokuyo Laser -->
   <link name="$(arg tf_prefix)/hokuyo">
@@ -39,11 +40,17 @@
     <parent link="$(arg tf_prefix)/base_sensors"/>
     <child link="$(arg tf_prefix)/xsens"/>
-    <origin xyz="0.05 0 0" rpy="0 0 0"/>
+    <origin xyz="-0.005 0 0" rpy="0 0 0"/>
   </joint>
-  <joint name="base_sens_hokuyo" type="fixed">
+   <joint name="base_sens_hokuyo" type="fixed">
     <parent link="$(arg tf_prefix)/base_sensors"/>
     <child link="$(arg tf_prefix)/hokuyo"/>
     <axis xyz="0 1 0" />
-    <origin xyz="0.0 0 0.09" rpy="0 0 0"/>
+    <origin xyz="0.08 0 0.01" rpy="0 0 0"/>
+  </joint>
+ <joint name="base_sens_velodyne" type="fixed">
+    <parent link="$(arg tf_prefix)/base_sensors"/>
+    <child link="$(arg tf_prefix)/velodyne"/>
+    <axis xyz="0 1 0" />
+    <origin xyz="-0.024 0 0.03" rpy="0 0 0"/>
   </joint>
   <!--hokuyo-->
