Commit message: Config files for thorvald_006

File: rasberry_bringup/urdf/robot_006_sensors.xacro (robot description, xacro)
@@ -3,7 +3,7 @@
   <xacro:arg name="robot_name" default=""/>
   <xacro:arg name="tf_prefix" default=""/>
-  <link name="$(arg tf_prefix)/base_sensors"/>
-  <link name="$(arg tf_prefix)/septentrio"/>
-  <link name="$(arg tf_prefix)/xsens"/>
+  <!--link name="$(arg tf_prefix)/base_sensors"/-->
+  <!--link name="$(arg tf_prefix)/septentrio"/-->
+  <!--link name="$(arg tf_prefix)/xsens"/-->
   <link name="$(arg tf_prefix)/velodyne"/>
   <!-- Hokuyo Laser -->
@@ -27,30 +27,30 @@
     </inertial>
   </link>
-  <joint name="base_base_sens" type="fixed">
+  <!--joint name="base_base_sens" type="fixed">
     <parent link="$(arg tf_prefix)/base_link"/>
     <child link="$(arg tf_prefix)/base_sensors"/>
     <origin xyz="0.547 0 0.77" rpy="0 0 0"/>
-  </joint>
-  <joint name="base_sens_septentrio" type="fixed">
+  </joint-->
+  <!--joint name="base_sens_septentrio" type="fixed">
     <parent link="$(arg tf_prefix)/base_sensors"/>
     <child link="$(arg tf_prefix)/septentrio"/>
     <origin xyz="-0.01 0 0.3" rpy="0 0 0"/>
-  </joint>
-  <joint name="base_sens_xsens" type="fixed">
+  </joint-->
+  <!--joint name="base_sens_xsens" type="fixed">
     <parent link="$(arg tf_prefix)/base_link"/>
     <child link="$(arg tf_prefix)/xsens"/>
     <origin xyz="0.018 0.258 0.69" rpy="0 0 0"/>
-  </joint>
+  </joint-->
    <joint name="base_sens_hokuyo" type="fixed">
     <parent link="$(arg tf_prefix)/base_link"/>
     <child link="$(arg tf_prefix)/hokuyo"/>
     <axis xyz="0 1 0" />
-    <origin xyz="0.7025 -0.0 0.66" rpy="3.141593 0.0 0.0"/>
+    <origin xyz="0.8305 -0.0 0.64" rpy="3.141593 0.0 0.0"/>
   </joint>
  <joint name="base_sens_velodyne" type="fixed">
-    <parent link="$(arg tf_prefix)/base_sensors"/>
+    <parent link="$(arg tf_prefix)/base_link"/>
     <child link="$(arg tf_prefix)/velodyne"/>
     <axis xyz="0 1 0" />
-    <origin xyz="-0.024 0 0.03" rpy="0 0 0"/>
+    <origin xyz="0.01 0 1.465" rpy="0 0 0"/>
   </joint>
   <!--hokuyo-->

Commit message: Updated robot sensor xacros IMUs disabled ROSBRIDGE_IP set to 10.8.0.18

File: rasberry_bringup/urdf/robot_006_sensors.xacro (robot description, xacro)
@@ -3,5 +3,5 @@
   <xacro:arg name="robot_name" default=""/>
   <xacro:arg name="tf_prefix" default=""/>
-  <!--link name="$(arg tf_prefix)/base_sensors"/-->
+  <link name="$(arg tf_prefix)/base_sensors"/>
   <!--link name="$(arg tf_prefix)/septentrio"/-->
   <!--link name="$(arg tf_prefix)/xsens"/-->
@@ -27,9 +27,9 @@
     </inertial>
   </link>
-  <!--joint name="base_base_sens" type="fixed">
+  <joint name="base_base_sens" type="fixed">
     <parent link="$(arg tf_prefix)/base_link"/>
     <child link="$(arg tf_prefix)/base_sensors"/>
-    <origin xyz="0.547 0 0.77" rpy="0 0 0"/>
-  </joint-->
+    <origin xyz="-0.370 -0.1075 1.440" rpy="0 0 0"/>
+  </joint>
   <!--joint name="base_sens_septentrio" type="fixed">
     <parent link="$(arg tf_prefix)/base_sensors"/>
@@ -46,11 +46,11 @@
     <child link="$(arg tf_prefix)/hokuyo"/>
     <axis xyz="0 1 0" />
-    <origin xyz="0.8305 -0.0 0.64" rpy="3.141593 0.0 0.0"/>
+    <origin xyz="0.8025 -0.0 0.65" rpy="3.141593 0.0 0.0"/>
   </joint>
  <joint name="base_sens_velodyne" type="fixed">
-    <parent link="$(arg tf_prefix)/base_link"/>
+    <parent link="$(arg tf_prefix)/base_sensors"/>
     <child link="$(arg tf_prefix)/velodyne"/>
     <axis xyz="0 1 0" />
-    <origin xyz="0.01 0 1.465" rpy="0 0 0"/>
+    <origin xyz="0.38 0.12 0.04" rpy="0 0 0"/>
   </joint>
   <!--hokuyo-->

File: rasberry_bringup/urdf/robot_007_sensors.xacro (robot description, xacro)
@@ -30,5 +30,5 @@
     <parent link="$(arg tf_prefix)/base_link"/>
     <child link="$(arg tf_prefix)/base_sensors"/>
-    <origin xyz="0.547 0 0.77" rpy="0 0 0"/>
+    <origin xyz="-0.370 -0.1075 1.440" rpy="0 0 0"/>
   </joint>
   <joint name="base_sens_septentrio" type="fixed">
@@ -52,5 +52,5 @@
     <child link="$(arg tf_prefix)/velodyne"/>
     <axis xyz="0 1 0" />
-    <origin xyz="-0.024 0 0.03" rpy="0 0 0"/>
+    <origin xyz="0.38 0.12 0.04" rpy="0 0 0"/>
   </joint>
   <!--hokuyo-->
