Commit message: Map, no go map and topological map added for the new simulation environment. The plant models have been removed (for now) from this world to speed the sim up. I will look at ways of increasing the sim's real-time factor that will allow me to put them back in. `rasberry_bringup/launch/hokuyo.launch` and `rasberry_bringup/urdf/robot_007_sensors.xacro` have been updated due to the adjustment of the yaw of the hokuyo on the physical robot (it is now at zero degrees).

File: rasberry_bringup/urdf/robot_007_sensors.xacro (robot description, xacro)
@@ -46,5 +46,5 @@
     <child link="$(arg tf_prefix)/hokuyo"/>
     <axis xyz="0 1 0" />
-    <origin xyz="0.7025 -0.0 0.66" rpy="3.14 0 -0.785"/>
+    <origin xyz="0.7025 -0.0 0.66" rpy="3.14 0.0 0.0"/>
   </joint>
  <joint name="base_sens_velodyne" type="fixed">
@@ -66,6 +66,6 @@
             <samples>720</samples>
             <resolution>1</resolution>
-            <min_angle>-2.356194</min_angle>
-            <max_angle>0.785398</max_angle>
+            <min_angle>-1.570796</min_angle>
+            <max_angle>1.570796</max_angle>
           </horizontal>
         </scan>

Commit message: Modifications to 007 config and sensor xacro

File: rasberry_bringup/urdf/robot_007_sensors.xacro (robot description, xacro)
@@ -40,5 +40,5 @@
     <parent link="$(arg tf_prefix)/base_link"/>
     <child link="$(arg tf_prefix)/xsens"/>
-    <origin xyz="0.018 0.258 0.69" rpy="0 0 0"/>
+    <origin xyz="-0.005 0.2605 0.682" rpy="0 0 0"/>
   </joint>
    <joint name="base_sens_hokuyo" type="fixed">
@@ -46,5 +46,5 @@
     <child link="$(arg tf_prefix)/hokuyo"/>
     <axis xyz="0 1 0" />
-    <origin xyz="0.7025 -0.0 0.66" rpy="3.141593 0.0 0.0"/>
+    <origin xyz="0.7025 0.005 0.66" rpy="3.141593 0.0 0.0"/>
   </joint>
  <joint name="base_sens_velodyne" type="fixed">

Commit message: thorvald 006 and 007 hostnames changed to 007 and 008 (as labelled on robot) respectively

File: rasberry_bringup/urdf/robot_007_sensors.xacro (robot description, xacro)
@@ -4,5 +4,5 @@
   <xacro:arg name="tf_prefix" default=""/>
   <link name="$(arg tf_prefix)/base_sensors"/>
-  <link name="$(arg tf_prefix)/septentrio"/>
+  <!--link name="$(arg tf_prefix)/septentrio"/-->
   <link name="$(arg tf_prefix)/xsens"/>
   <link name="$(arg tf_prefix)/velodyne"/>
@@ -30,15 +30,16 @@
     <parent link="$(arg tf_prefix)/base_link"/>
     <child link="$(arg tf_prefix)/base_sensors"/>
-    <origin xyz="-0.370 -0.1075 1.440" rpy="0 0 0"/>
+    <!-- <origin xyz="-0.370 -0.1075 1.440" rpy="0 0 0"/> -->
+    <origin xyz="-0.370 -0.115 1.440" rpy="0 0 0"/>
   </joint>
-  <joint name="base_sens_septentrio" type="fixed">
+  <!--joint name="base_sens_septentrio" type="fixed">
     <parent link="$(arg tf_prefix)/base_sensors"/>
     <child link="$(arg tf_prefix)/septentrio"/>
     <origin xyz="-0.01 0 0.3" rpy="0 0 0"/>
-  </joint>
+  </joint-->
   <joint name="base_sens_xsens" type="fixed">
     <parent link="$(arg tf_prefix)/base_link"/>
     <child link="$(arg tf_prefix)/xsens"/>
-    <origin xyz="-0.005 0.2605 0.682" rpy="0 0 0"/>
+    <origin xyz="0.8025 -0.05 0.76" rpy="0 0 0"/>
   </joint>
    <joint name="base_sens_hokuyo" type="fixed">
@@ -46,5 +47,5 @@
     <child link="$(arg tf_prefix)/hokuyo"/>
     <axis xyz="0 1 0" />
-    <origin xyz="0.7025 0.005 0.66" rpy="3.141593 0.0 0.0"/>
+    <origin xyz="0.8025 -0.0 0.65" rpy="3.141593 0.0 0.0"/>
   </joint>
  <joint name="base_sens_velodyne" type="fixed">
@@ -52,5 +53,17 @@
     <child link="$(arg tf_prefix)/velodyne"/>
     <axis xyz="0 1 0" />
-    <origin xyz="0.38 0.12 0.04" rpy="0 0 0"/>
+    <origin xyz="0.38 -0.122 0.04" rpy="0 0 0"/>
+  </joint>
+ <joint name="base_sens_thermal" type="fixed">
+    <parent link="$(arg tf_prefix)/base_sensors"/>
+    <child link="$(arg tf_prefix)/thermal_camera"/>
+    <axis xyz="0 1 0" />
+    <origin xyz="0.29 0.135 0.115" rpy="0 0 0"/>
+  </joint>
+ <joint name="base_sens_kinect2" type="fixed">
+    <parent link="$(arg tf_prefix)/base_sensors"/>
+    <child link="$(arg tf_prefix)/kinect2_color_camera"/>
+    <axis xyz="0 1 0" />
+    <origin xyz="0.494 0.0025 0.023" rpy="0 0 0"/>
   </joint>
   <!--hokuyo-->

File: rasberry_bringup/urdf/robot_008_sensors.xacro (robot description, xacro)
@@ -4,6 +4,6 @@
   <xacro:arg name="tf_prefix" default=""/>
   <link name="$(arg tf_prefix)/base_sensors"/>
-  <!--link name="$(arg tf_prefix)/septentrio"/-->
-  <!--link name="$(arg tf_prefix)/xsens"/-->
+  <link name="$(arg tf_prefix)/septentrio"/>
+  <link name="$(arg tf_prefix)/xsens"/>
   <link name="$(arg tf_prefix)/velodyne"/>
   <!-- Hokuyo Laser -->
@@ -32,19 +32,19 @@
     <origin xyz="-0.370 -0.1075 1.440" rpy="0 0 0"/>
   </joint>
-  <!--joint name="base_sens_septentrio" type="fixed">
+  <joint name="base_sens_septentrio" type="fixed">
     <parent link="$(arg tf_prefix)/base_sensors"/>
     <child link="$(arg tf_prefix)/septentrio"/>
     <origin xyz="-0.01 0 0.3" rpy="0 0 0"/>
-  </joint-->
-  <!--joint name="base_sens_xsens" type="fixed">
+  </joint>
+  <joint name="base_sens_xsens" type="fixed">
     <parent link="$(arg tf_prefix)/base_link"/>
     <child link="$(arg tf_prefix)/xsens"/>
-    <origin xyz="0.018 0.258 0.69" rpy="0 0 0"/>
-  </joint-->
+    <origin xyz="-0.005 0.2605 0.682" rpy="0 0 0"/>
+  </joint>
    <joint name="base_sens_hokuyo" type="fixed">
     <parent link="$(arg tf_prefix)/base_link"/>
     <child link="$(arg tf_prefix)/hokuyo"/>
     <axis xyz="0 1 0" />
-    <origin xyz="0.8025 -0.0 0.65" rpy="3.141593 0.0 0.0"/>
+    <origin xyz="0.7025 0.005 0.66" rpy="3.141593 0.0 0.0"/>
   </joint>
  <joint name="base_sens_velodyne" type="fixed">
@@ -52,5 +52,5 @@
     <child link="$(arg tf_prefix)/velodyne"/>
     <axis xyz="0 1 0" />
-    <origin xyz="0.38 0.12 0.04" rpy="0 0 0"/>
+    <origin xyz="0.38 -0.122 0.04" rpy="0 0 0"/>
   </joint>
   <!--hokuyo-->

Commit message: missing links added in robot_007_sensors.xacro

File: rasberry_bringup/urdf/robot_007_sensors.xacro (robot description, xacro)
@@ -7,4 +7,6 @@
   <link name="$(arg tf_prefix)/xsens"/>
   <link name="$(arg tf_prefix)/velodyne"/>
+  <link name="$(arg tf_prefix)/thermal_camera"/>
+  <link name="$(arg tf_prefix)/kinect2_color_camera"/>"
   <!-- Hokuyo Laser -->
   <link name="$(arg tf_prefix)/hokuyo">

Commit message: Fixed wrong kinect2 tf frame name

File: rasberry_bringup/urdf/robot_007_sensors.xacro (robot description, xacro)
@@ -8,5 +8,5 @@
   <link name="$(arg tf_prefix)/velodyne"/>
   <link name="$(arg tf_prefix)/thermal_camera"/>
-  <link name="$(arg tf_prefix)/kinect2_color_camera"/>"
+  <link name="$(arg tf_prefix)/kinect2_rgb_optical_frame"/>"
   <!-- Hokuyo Laser -->
   <link name="$(arg tf_prefix)/hokuyo">
@@ -65,5 +65,5 @@
  <joint name="base_sens_kinect2" type="fixed">
     <parent link="$(arg tf_prefix)/base_sensors"/>
-    <child link="$(arg tf_prefix)/kinect2_color_camera"/>
+    <child link="$(arg tf_prefix)/kinect2_rgb_optical_frame"/>
     <axis xyz="0 1 0" />
     <origin xyz="0.494 0.0025 0.023" rpy="0 0 0"/>
