Commit message: amcl optimisation capability added to `rasberry_optimise` package. New amcl params added for testing.

File: rasberry_bringup/urdf/robot_008_sensors.xacro (robot description, xacro)
@@ -46,5 +46,5 @@
     <child link="$(arg tf_prefix)/hokuyo"/>
     <axis xyz="0 1 0" />
-    <origin xyz="0.7025 0.005 0.66" rpy="3.141593 0.0 0.0"/>
+    <origin xyz="0.7025 0.0 0.66" rpy="3.141593 0.0 0.0"/>
   </joint>
  <joint name="base_sens_velodyne" type="fixed">
@@ -82,5 +82,5 @@
                reading. -->
           <mean>0.0</mean>
-          <stddev>0.01</stddev>
+          <stddev>0.05</stddev>
         </noise>
       </ray>
