Commit message: thorvald_model -> thorvald_description

File: rasberry_bringup/urdf/robot_003_sensors.xacro (robot description, xacro)
@@ -18,5 +18,5 @@
       <origin xyz="0 0 0" rpy="0 0 0"/>
       <geometry>
-        <mesh filename="package://thorvald_model/meshes/hokuyo/hokuyo.dae"/>
+        <mesh filename="package://thorvald_description/meshes/hokuyo/hokuyo.dae"/>
       </geometry>
     </visual>

File: rasberry_bringup/urdf/robot_005_sensors.xacro (robot description, xacro)
@@ -18,5 +18,5 @@
       <origin xyz="0 0 0" rpy="0 0 0"/>
       <geometry>
-        <mesh filename="package://thorvald_model/meshes/hokuyo/hokuyo.dae"/>
+        <mesh filename="package://thorvald_description/meshes/hokuyo/hokuyo.dae"/>
       </geometry>
     </visual>

File: rasberry_bringup/urdf/robot_007_sensors.xacro (robot description, xacro)
@@ -20,5 +20,5 @@
       <origin xyz="0 0 0" rpy="0 0 0"/>
       <geometry>
-        <mesh filename="package://thorvald_model/meshes/hokuyo/hokuyo.dae"/>
+        <mesh filename="package://thorvald_description/meshes/hokuyo/hokuyo.dae"/>
       </geometry>
     </visual>

File: rasberry_bringup/urdf/robot_008_sensors.xacro (robot description, xacro)
@@ -18,5 +18,5 @@
       <origin xyz="0 0 0" rpy="0 0 0"/>
       <geometry>
-        <mesh filename="package://thorvald_model/meshes/hokuyo/hokuyo.dae"/>
+        <mesh filename="package://thorvald_description/meshes/hokuyo/hokuyo.dae"/>
       </geometry>
     </visual>

File: rasberry_bringup/urdf/robot_008_sensors_corner_hokuyos.xacro (robot description, xacro)
@@ -18,5 +18,5 @@
       <origin xyz="0 0 0" rpy="0 0 0"/>
       <geometry>
-        <mesh filename="package://thorvald_model/meshes/hokuyo/hokuyo.dae"/>
+        <mesh filename="package://thorvald_description/meshes/hokuyo/hokuyo.dae"/>
       </geometry>
     </visual>
@@ -38,5 +38,5 @@
       <origin xyz="0 0 0" rpy="0 0 0"/>
       <geometry>
-        <mesh filename="package://thorvald_model/meshes/hokuyo/hokuyo.dae"/>
+        <mesh filename="package://thorvald_description/meshes/hokuyo/hokuyo.dae"/>
       </geometry>
     </visual>

File: rasberry_bringup/urdf/robot_014_sensors.xacro (robot description, xacro)
@@ -18,5 +18,5 @@
       <origin xyz="0 0 0" rpy="0 0 0"/>
       <geometry>
-        <mesh filename="package://thorvald_model/meshes/hokuyo/hokuyo.dae"/>
+        <mesh filename="package://thorvald_description/meshes/hokuyo/hokuyo.dae"/>
       </geometry>
     </visual>

File: rasberry_bringup/urdf/robot_014_sensors_corner_hokuyos.xacro (robot description, xacro)
@@ -18,5 +18,5 @@
       <origin xyz="0 0 0" rpy="0 0 0"/>
       <geometry>
-        <mesh filename="package://thorvald_model/meshes/hokuyo/hokuyo.dae"/>
+        <mesh filename="package://thorvald_description/meshes/hokuyo/hokuyo.dae"/>
       </geometry>
     </visual>
@@ -38,5 +38,5 @@
       <origin xyz="0 0 0" rpy="0 0 0"/>
       <geometry>
-        <mesh filename="package://thorvald_model/meshes/hokuyo/hokuyo.dae"/>
+        <mesh filename="package://thorvald_description/meshes/hokuyo/hokuyo.dae"/>
       </geometry>
     </visual>
