Commit message: hokuyos are assumed to be in the correct upside up
sensors xacro updated

File: rasberry_bringup/urdf/robot_008_sensors_corner_hokuyos.xacro (robot description, xacro)
@@ -66,5 +66,5 @@
     <child link="$(arg tf_prefix)/hokuyo_fr"/>
     <axis xyz="0 1 0" />
-    <origin xyz="0.6959 -0.4835 0.59" rpy="3.141593 0.0 -0.79"/>
+    <origin xyz="0.704 -0.439 0.705" rpy="0.0 0.0 -0.79"/>
   </joint>
    <joint name="base_sens_hokuyo_bl" type="fixed">
@@ -72,5 +72,5 @@
     <child link="$(arg tf_prefix)/hokuyo_bl"/>
     <axis xyz="0 1 0" />
-    <origin xyz="-0.6959 0.4835 0.59" rpy="3.141593 0.0 2.36"/>
+    <origin xyz="-0.704 0.439 0.705" rpy="0.0 0.0 2.36"/>
   </joint>
  <joint name="base_sens_velodyne" type="fixed">

Commit message: 1. removed corner reference in the hokuyo positions   - _fl (front-left) now changed to _front   - _br (back-right) now changed to _back   - same conventions for hokuyo_xx frames, scan_xx topics 2. hokuyo position corrected to new bracket positions

File: rasberry_bringup/urdf/robot_008_sensors_corner_hokuyos.xacro (robot description, xacro)
@@ -8,5 +8,5 @@
   <link name="$(arg tf_prefix)/velodyne"/>
   <!-- Hokuyo Laser -->
-  <link name="$(arg tf_prefix)/hokuyo_fl">
+  <link name="$(arg tf_prefix)/hokuyo_front">
     <collision>
       <origin xyz="0 0 0" rpy="0 0 0"/>
@@ -28,5 +28,5 @@
   </link>
  <!-- Hokuyo Laser -->
-  <link name="$(arg tf_prefix)/hokuyo_br">
+  <link name="$(arg tf_prefix)/hokuyo_back">
     <collision>
       <origin xyz="0 0 0" rpy="0 0 0"/>
@@ -62,13 +62,13 @@
     <origin xyz="-0.005 0.2605 0.682" rpy="0 0 0"/>
   </joint>
-   <joint name="base_sens_hokuyo_fl" type="fixed">
+   <joint name="base_sens_hokuyo_front" type="fixed">
     <parent link="$(arg tf_prefix)/base_link"/>
-    <child link="$(arg tf_prefix)/hokuyo_fl"/>
+    <child link="$(arg tf_prefix)/hokuyo_front"/>
     <axis xyz="0 1 0" />
     <origin xyz="0.700 0.485 0.705" rpy="0.0 0.0 0.79"/>
   </joint>
-   <joint name="base_sens_hokuyo_br" type="fixed">
+   <joint name="base_sens_hokuyo_back" type="fixed">
     <parent link="$(arg tf_prefix)/base_link"/>
-    <child link="$(arg tf_prefix)/hokuyo_br"/>
+    <child link="$(arg tf_prefix)/hokuyo_back"/>
     <axis xyz="0 1 0" />
     <origin xyz="-0.700 -0.485 0.705" rpy="0.0 0.0 -2.36"/>
@@ -81,6 +81,6 @@
   </joint>
   <!--hokuyo-->
-  <gazebo reference="$(arg tf_prefix)/hokuyo_fl">
-    <sensor name="$(arg robot_name)_head_hokuyo_fl_sensor" type="ray">
+  <gazebo reference="$(arg tf_prefix)/hokuyo_front">
+    <sensor name="$(arg robot_name)_head_hokuyo_front_sensor" type="ray">
       <pose>0 0 0 0 0 0</pose>
       <visualize>true</visualize>
@@ -111,13 +111,13 @@
         </noise>
       </ray>
-      <plugin name="$(arg robot_name)_hokuyo_fl_node" filename="libgazebo_ros_laser.so">
-        <topicName>scan_fl</topicName>
-        <frameName>hokuyo_fl</frameName>
+      <plugin name="$(arg robot_name)_hokuyo_front_node" filename="libgazebo_ros_laser.so">
+        <topicName>scan_front</topicName>
+        <frameName>hokuyo_front</frameName>
       </plugin>
     </sensor>
   </gazebo>
   <!--hokuyo-->
-  <gazebo reference="$(arg tf_prefix)/hokuyo_br">
-    <sensor name="$(arg robot_name)_head_hokuyo_br_sensor" type="ray">
+  <gazebo reference="$(arg tf_prefix)/hokuyo_back">
+    <sensor name="$(arg robot_name)_head_hokuyo_back_sensor" type="ray">
       <pose>0 0 0 0 0 0</pose>
       <visualize>true</visualize>
@@ -148,7 +148,7 @@
         </noise>
       </ray>
-      <plugin name="$(arg robot_name)_hokuyo_br_node" filename="libgazebo_ros_laser.so">
-        <topicName>scan_br</topicName>
-        <frameName>hokuyo_br</frameName>
+      <plugin name="$(arg robot_name)_hokuyo_back_node" filename="libgazebo_ros_laser.so">
+        <topicName>scan_back</topicName>
+        <frameName>hokuyo_back</frameName>
       </plugin>
     </sensor>

File: rasberry_bringup/urdf/robot_014_sensors_corner_hokuyos.xacro (robot description, xacro)
@@ -8,5 +8,5 @@
   <link name="$(arg tf_prefix)/velodyne"/>
   <!-- Hokuyo Laser -->
-  <link name="$(arg tf_prefix)/hokuyo_fl">
+  <link name="$(arg tf_prefix)/hokuyo_front">
     <collision>
       <origin xyz="0 0 0" rpy="0 0 0"/>
@@ -28,5 +28,5 @@
   </link>
  <!-- Hokuyo Laser -->
-  <link name="$(arg tf_prefix)/hokuyo_br">
+  <link name="$(arg tf_prefix)/hokuyo_back">
     <collision>
       <origin xyz="0 0 0" rpy="0 0 0"/>
@@ -62,15 +62,15 @@
     <origin xyz="-0.005 0.2605 0.682" rpy="0 0 0"/>
   </joint>
-   <joint name="base_sens_hokuyo_fl" type="fixed">
+   <joint name="base_sens_hokuyo_front" type="fixed">
     <parent link="$(arg tf_prefix)/base_link"/>
-    <child link="$(arg tf_prefix)/hokuyo_fl"/>
+    <child link="$(arg tf_prefix)/hokuyo_front"/>
     <axis xyz="0 1 0" />
-    <origin xyz="0.704 0.430 0.685" rpy="3.14 0.0 0.79"/>
+    <origin xyz="0.719 -0.433 0.640" rpy="0.0 0.0 -0.79"/>
   </joint>
-   <joint name="base_sens_hokuyo_br" type="fixed">
+   <joint name="base_sens_hokuyo_back" type="fixed">
     <parent link="$(arg tf_prefix)/base_link"/>
-    <child link="$(arg tf_prefix)/hokuyo_br"/>
+    <child link="$(arg tf_prefix)/hokuyo_back"/>
     <axis xyz="0 1 0" />
-    <origin xyz="-0.704 -0.430 0.705" rpy="3.14 0.0 -2.36"/>
+    <origin xyz="-0.719 0.433 0.640" rpy="0.0 0.0 2.36"/>
   </joint>
  <joint name="base_sens_velodyne" type="fixed">
@@ -81,6 +81,6 @@
   </joint>
   <!--hokuyo-->
-  <gazebo reference="$(arg tf_prefix)/hokuyo_fl">
-    <sensor name="$(arg robot_name)_head_hokuyo_fl_sensor" type="ray">
+  <gazebo reference="$(arg tf_prefix)/hokuyo_front">
+    <sensor name="$(arg robot_name)_head_hokuyo_front_sensor" type="ray">
       <pose>0 0 0 0 0 0</pose>
       <visualize>true</visualize>
@@ -111,13 +111,13 @@
         </noise>
       </ray>
-      <plugin name="$(arg robot_name)_hokuyo_fl_node" filename="libgazebo_ros_laser.so">
-        <topicName>scan_fl</topicName>
-        <frameName>hokuyo_fl</frameName>
+      <plugin name="$(arg robot_name)_hokuyo_front_node" filename="libgazebo_ros_laser.so">
+        <topicName>scan_front</topicName>
+        <frameName>hokuyo_front</frameName>
       </plugin>
     </sensor>
   </gazebo>
   <!--hokuyo-->
-  <gazebo reference="$(arg tf_prefix)/hokuyo_br">
-    <sensor name="$(arg robot_name)_head_hokuyo_br_sensor" type="ray">
+  <gazebo reference="$(arg tf_prefix)/hokuyo_back">
+    <sensor name="$(arg robot_name)_head_hokuyo_back_sensor" type="ray">
       <pose>0 0 0 0 0 0</pose>
       <visualize>true</visualize>
@@ -148,7 +148,7 @@
         </noise>
       </ray>
-      <plugin name="$(arg robot_name)_hokuyo_br_node" filename="libgazebo_ros_laser.so">
-        <topicName>scan_br</topicName>
-        <frameName>hokuyo_br</frameName>
+      <plugin name="$(arg robot_name)_hokuyo_back_node" filename="libgazebo_ros_laser.so">
+        <topicName>scan_back</topicName>
+        <frameName>hokuyo_back</frameName>
       </plugin>
     </sensor>

Commit message: First working verion of multisim and des pickers
Summary:
1. DES pickers + real pickers detected by marvelmind
2. DES runs in realtime mode and DES pickers calls the service to add task whenever the tray_full event happens for each of them.
3. DES pickers' calls and real pickers' calls are serviced by rasberry_coordinator - So no descriminition between the two.
4. This sim exclusively uses robots with corner hokuyos and expects bidirectional topo maps

Known issues:
1. Only one iteration of picking is implemented now
2. multi-robot traffic blocks in topo_nav yet to be solved

Changes:
1. rosparam correction in robot_bringup_multisim.launch
2. rviz configuration updates
3. corner_hokuyos sensor xacro adjustments for 008 and hokuyo angles for 014
4. DES' mimic version of files work with with_robots = True/False cases
5. minor name changes in costmap_common_params_corner_hokuyos.yaml

File: rasberry_bringup/urdf/robot_008_sensors_corner_hokuyos.xacro (robot description, xacro)
@@ -53,12 +53,12 @@
   </joint>
   <joint name="base_sens_septentrio" type="fixed">
-    <parent link="$(arg tf_prefix)/base_sensors"/>
+    <parent link="$(arg tf_prefix)/base_link"/>
     <child link="$(arg tf_prefix)/septentrio"/>
-    <origin xyz="-0.01 0 0.3" rpy="0 0 0"/>
+    <origin xyz="-0.5325 -0.314 0.814" rpy="0 0 0"/>
   </joint>
   <joint name="base_sens_xsens" type="fixed">
     <parent link="$(arg tf_prefix)/base_link"/>
     <child link="$(arg tf_prefix)/xsens"/>
-    <origin xyz="-0.005 0.2605 0.682" rpy="0 0 0"/>
+    <origin xyz="0.18 -0.266 0.717" rpy="0 0 0"/>
   </joint>
    <joint name="base_sens_hokuyo_front" type="fixed">
@@ -66,5 +66,5 @@
     <child link="$(arg tf_prefix)/hokuyo_front"/>
     <axis xyz="0 1 0" />
-    <origin xyz="0.700 0.485 0.705" rpy="0.0 0.0 0.79"/>
+    <origin xyz="0.719 -0.433 0.640" rpy="0.0 0.0 -0.79"/>
   </joint>
    <joint name="base_sens_hokuyo_back" type="fixed">
@@ -72,5 +72,5 @@
     <child link="$(arg tf_prefix)/hokuyo_back"/>
     <axis xyz="0 1 0" />
-    <origin xyz="-0.700 -0.485 0.705" rpy="0.0 0.0 -2.36"/>
+    <origin xyz="-0.719 0.433 0.640" rpy="0.0 0.0 2.36"/>
   </joint>
  <joint name="base_sens_velodyne" type="fixed">
@@ -92,6 +92,6 @@
             <samples>720</samples>
             <resolution>1</resolution>
-            <min_angle>-2.36</min_angle>
-            <max_angle>2.36</max_angle>
+            <min_angle>-2.18</min_angle>
+            <max_angle>2.18</max_angle>
           </horizontal>
         </scan>
@@ -129,6 +129,6 @@
             <samples>720</samples>
             <resolution>1</resolution>
-            <min_angle>-2.36</min_angle>
-            <max_angle>2.36</max_angle>
+            <min_angle>-2.18</min_angle>
+            <max_angle>2.18</max_angle>
           </horizontal>
         </scan>

File: rasberry_bringup/urdf/robot_014_sensors_corner_hokuyos.xacro (robot description, xacro)
@@ -93,5 +93,5 @@
             <resolution>1</resolution>
             <min_angle>-2.18</min_angle>
-            <max_angle>2.36</max_angle>
+            <max_angle>2.18</max_angle>
           </horizontal>
         </scan>
@@ -130,5 +130,5 @@
             <resolution>1</resolution>
             <min_angle>-2.18</min_angle>
-            <max_angle>2.36</max_angle>
+            <max_angle>2.18</max_angle>
           </horizontal>
         </scan>

Commit message: Update xacro files for new sensor racks

File: rasberry_bringup/urdf/robot_008_sensors_corner_hokuyos.xacro (robot description, xacro)
@@ -50,5 +50,5 @@
     <parent link="$(arg tf_prefix)/base_link"/>
     <child link="$(arg tf_prefix)/base_sensors"/>
-    <origin xyz="-0.370 -0.1075 1.440" rpy="0 0 0"/>
+    <origin xyz="0 0 1.52" rpy="0 0 0"/>
   </joint>
   <joint name="base_sens_septentrio" type="fixed">
@@ -60,5 +60,5 @@
     <parent link="$(arg tf_prefix)/base_link"/>
     <child link="$(arg tf_prefix)/xsens"/>
-    <origin xyz="-0.005 0.2605 0.682" rpy="0 0 0"/>
+    <origin xyz="0.18 -0.266 0.717" rpy="0 0 0"/>
   </joint>
    <joint name="base_sens_hokuyo_front" type="fixed">
@@ -66,5 +66,5 @@
     <child link="$(arg tf_prefix)/hokuyo_front"/>
     <axis xyz="0 1 0" />
-    <origin xyz="0.700 0.485 0.705" rpy="0.0 0.0 0.79"/>
+    <origin xyz="0.719 -0.433 0.640" rpy="0.0 0.0 -0.79"/>
   </joint>
    <joint name="base_sens_hokuyo_back" type="fixed">
@@ -72,5 +72,5 @@
     <child link="$(arg tf_prefix)/hokuyo_back"/>
     <axis xyz="0 1 0" />
-    <origin xyz="-0.700 -0.485 0.705" rpy="0.0 0.0 -2.36"/>
+    <origin xyz="-0.719 0.433 0.640" rpy="0.0 0.0 2.36"/>
   </joint>
  <joint name="base_sens_velodyne" type="fixed">
@@ -78,5 +78,5 @@
     <child link="$(arg tf_prefix)/velodyne"/>
     <axis xyz="0 1 0" />
-    <origin xyz="0.38 -0.122 0.04" rpy="0 0 0"/>
+    <origin xyz="0 0 0" rpy="0 0 0"/>
   </joint>
   <!--hokuyo-->
@@ -92,5 +92,5 @@
             <samples>720</samples>
             <resolution>1</resolution>
-            <min_angle>-2.36</min_angle>
+            <min_angle>-2.18</min_angle>
             <max_angle>2.36</max_angle>
           </horizontal>
@@ -129,5 +129,5 @@
             <samples>720</samples>
             <resolution>1</resolution>
-            <min_angle>-2.36</min_angle>
+            <min_angle>-2.18</min_angle>
             <max_angle>2.36</max_angle>
           </horizontal>

File: rasberry_bringup/urdf/robot_014_sensors_corner_hokuyos.xacro (robot description, xacro)
@@ -50,5 +50,5 @@
     <parent link="$(arg tf_prefix)/base_link"/>
     <child link="$(arg tf_prefix)/base_sensors"/>
-    <origin xyz="-0.370 -0.1075 1.440" rpy="0 0 0"/>
+    <origin xyz="0 0 1.52" rpy="0 0 0"/>
   </joint>
   <joint name="base_sens_septentrio" type="fixed">
@@ -78,5 +78,5 @@
     <child link="$(arg tf_prefix)/velodyne"/>
     <axis xyz="0 1 0" />
-    <origin xyz="0.38 -0.122 0.04" rpy="0 0 0"/>
+    <origin xyz="0 0 0" rpy="0 0 0"/>
   </joint>
   <!--hokuyo-->

Commit message: joint position of back hokuyo is corrected
joint position of back hokuyo is corrected on 15 wrt top3. earlier the laser position was inside the robot.
robot 008 and 014's corner_hokuyos sensor xacros are also modified to match 15's way of hokuyo joint positions wrt to `top` frames.

File: rasberry_bringup/urdf/robot_008_sensors_corner_hokuyos.xacro (robot description, xacro)
@@ -63,14 +63,14 @@
   </joint>
    <joint name="base_sens_hokuyo_front" type="fixed">
-    <parent link="$(arg tf_prefix)/base_link"/>
+    <parent link="$(arg tf_prefix)/top1"/>
     <child link="$(arg tf_prefix)/hokuyo_front"/>
     <axis xyz="0 1 0" />
-    <origin xyz="0.719 -0.433 0.640" rpy="0.0 0.0 -0.79"/>
+    <origin xyz="0.172 -0.152 -0.034" rpy="0.0 0.0 -0.79"/>
   </joint>
    <joint name="base_sens_hokuyo_back" type="fixed">
-    <parent link="$(arg tf_prefix)/base_link"/>
+    <parent link="$(arg tf_prefix)/top3"/>
     <child link="$(arg tf_prefix)/hokuyo_back"/>
     <axis xyz="0 1 0" />
-    <origin xyz="-0.719 0.433 0.640" rpy="0.0 0.0 2.36"/>
+    <origin xyz="0.172 -0.152 -0.034" rpy="0.0 0.0 -0.79"/>
   </joint>
  <joint name="base_sens_velodyne" type="fixed">

File: rasberry_bringup/urdf/robot_014_sensors_corner_hokuyos.xacro (robot description, xacro)
@@ -63,14 +63,14 @@
   </joint>
    <joint name="base_sens_hokuyo_front" type="fixed">
-    <parent link="$(arg tf_prefix)/base_link"/>
+    <parent link="$(arg tf_prefix)/top1"/>
     <child link="$(arg tf_prefix)/hokuyo_front"/>
     <axis xyz="0 1 0" />
-    <origin xyz="0.719 -0.433 0.640" rpy="0.0 0.0 -0.79"/>
+    <origin xyz="0.172 -0.152 -0.034" rpy="0.0 0.0 -0.79"/>
   </joint>
    <joint name="base_sens_hokuyo_back" type="fixed">
-    <parent link="$(arg tf_prefix)/base_link"/>
+    <parent link="$(arg tf_prefix)/top3"/>
     <child link="$(arg tf_prefix)/hokuyo_back"/>
     <axis xyz="0 1 0" />
-    <origin xyz="-0.719 0.433 0.640" rpy="0.0 0.0 2.36"/>
+    <origin xyz="0.172 -0.152 -0.034" rpy="0.0 0.0 -0.79"/>
   </joint>
  <joint name="base_sens_velodyne" type="fixed">
@@ -93,5 +93,5 @@
             <resolution>1</resolution>
             <min_angle>-2.18</min_angle>
-            <max_angle>2.18</max_angle>
+            <max_angle>2.36</max_angle>
           </horizontal>
         </scan>
@@ -130,5 +130,5 @@
             <resolution>1</resolution>
             <min_angle>-2.18</min_angle>
-            <max_angle>2.18</max_angle>
+            <max_angle>2.36</max_angle>
           </horizontal>
         </scan>

File: rasberry_bringup/urdf/robot_015_sensors_corner_hokuyos.xacro (robot description, xacro)
@@ -66,5 +66,5 @@
     <child link="$(arg tf_prefix)/hokuyo_front"/>
     <axis xyz="0 1 0" />
-    <origin xyz="0.172 -0.152 0.034" rpy="0.0 0.0 -0.79"/>
+    <origin xyz="0.172 -0.152 -0.034" rpy="0.0 0.0 -0.79"/>
   </joint>
    <joint name="base_sens_hokuyo_back" type="fixed">
@@ -72,5 +72,5 @@
     <child link="$(arg tf_prefix)/hokuyo_back"/>
     <axis xyz="0 1 0" />
-    <origin xyz="-0.172 0.152 0.034" rpy="0.0 0.0 2.36"/>
+    <origin xyz="0.172 -0.152 -0.034" rpy="0.0 0.0 -0.79"/>
   </joint>
  <joint name="base_sens_velodyne" type="fixed">
