Commit message: fixed reference frame of back_hokuyos frame from top2 to top3

File: rasberry_bringup/urdf/robot_015_sensors_corner_hokuyos.xacro (robot description, xacro)
@@ -69,5 +69,5 @@
   </joint>
    <joint name="base_sens_hokuyo_back" type="fixed">
-    <parent link="$(arg tf_prefix)/top2"/>
+    <parent link="$(arg tf_prefix)/top3"/>
     <child link="$(arg tf_prefix)/hokuyo_back"/>
     <axis xyz="0 1 0" />

Commit message: New xacro for thorvald-015 (#309)

File: rasberry_bringup/urdf/robot_015_sensors_corner_hokuyos.xacro (robot description, xacro)
@@ -78,5 +78,5 @@
     <child link="$(arg tf_prefix)/velodyne"/>
     <axis xyz="0 1 0" />
-    <origin xyz="0 0 0" rpy="0 0 0"/>
+    <origin xyz="0 0 0" rpy="0 0 3.14159"/>
   </joint>
   <!--hokuyo-->
