Commit message: add um7 to 14 urdf

File: rasberry_bringup/urdf/robot_014_sensors.xacro (robot description, xacro)
@@ -41,4 +41,9 @@
     <child link="$(arg tf_prefix)/xsens"/>
     <origin xyz="-0.005 0.2605 0.682" rpy="0 0 0"/>
+  </joint>
+  <joint name="base_sens_um7" type="fixed">
+    <parent link="$(arg tf_prefix)/base_link"/>
+    <child link="$(arg tf_prefix)/imu_link"/>
+    <origin xyz="0.20 0.16 0.69" rpy="0 0 0"/>
   </joint>
    <joint name="base_sens_hokuyo" type="fixed">

Commit message: adjust xsens in 14 urdf

File: rasberry_bringup/urdf/robot_014_sensors.xacro (robot description, xacro)
@@ -40,5 +40,5 @@
     <parent link="$(arg tf_prefix)/base_link"/>
     <child link="$(arg tf_prefix)/xsens"/>
-    <origin xyz="-0.005 0.2605 0.682" rpy="0 0 0"/>
+    <origin xyz="0.00 -0.23 0.69" rpy="0 0 0"/>
   </joint>
   <joint name="base_sens_um7" type="fixed">

Commit message: adjust xsens in 14 & 19 urdf

File: rasberry_bringup/urdf/robot_014_sensors.xacro (robot description, xacro)
@@ -40,10 +40,5 @@
     <parent link="$(arg tf_prefix)/base_link"/>
     <child link="$(arg tf_prefix)/xsens"/>
-    <origin xyz="0.00 -0.23 0.69" rpy="0 0 0"/>
-  </joint>
-  <joint name="base_sens_um7" type="fixed">
-    <parent link="$(arg tf_prefix)/base_link"/>
-    <child link="$(arg tf_prefix)/imu_link"/>
-    <origin xyz="0.20 0.16 0.69" rpy="0 0 0"/>
+    <origin xyz="-0.005 0.2605 0.682" rpy="0 0 0"/>
   </joint>
    <joint name="base_sens_hokuyo" type="fixed">

File: rasberry_bringup/urdf/robot_014_sensors_corner_hokuyos.xacro (robot description, xacro)
@@ -60,5 +60,5 @@
     <parent link="$(arg tf_prefix)/base_link"/>
     <child link="$(arg tf_prefix)/xsens"/>
-    <origin xyz="0.18 -0.266 0.717" rpy="0 0 0"/>
+    <origin xyz="0.00 -0.23 0.69" rpy="0 0 0"/>
   </joint>
   <joint name="base_sens_um7" type="fixed">

File: rasberry_bringup/urdf/robot_019_sensors_corner_hokuyos.xacro (robot description, xacro)
@@ -60,5 +60,5 @@
     <parent link="$(arg tf_prefix)/base_link"/>
     <child link="$(arg tf_prefix)/xsens"/>
-    <origin xyz="0.18 -0.266 0.717" rpy="0 0 0"/>
+    <origin xyz="0.00 -0.23 0.69" rpy="0 0 0"/>
   </joint>
   <joint name="base_sens_um7" type="fixed">
