Commit message: hokuyo orientation corrected

File: rasberry_bringup/urdf/robot_014_sensors_corner_hokuyos.xacro (robot description, xacro)
@@ -66,5 +66,5 @@
     <child link="$(arg tf_prefix)/hokuyo_fl"/>
     <axis xyz="0 1 0" />
-    <origin xyz="0.700 0.485 0.705" rpy="0.0 0.0 0.79"/>
+    <origin xyz="0.704 0.430 0.685" rpy="3.14 0.0 0.79"/>
   </joint>
    <joint name="base_sens_hokuyo_br" type="fixed">
@@ -72,5 +72,5 @@
     <child link="$(arg tf_prefix)/hokuyo_br"/>
     <axis xyz="0 1 0" />
-    <origin xyz="-0.700 -0.485 0.705" rpy="0.0 0.0 -2.36"/>
+    <origin xyz="-0.704 -0.430 0.705" rpy="3.14 0.0 -2.36"/>
   </joint>
  <joint name="base_sens_velodyne" type="fixed">

Commit message: 014 xacro updates and hokuyo ips in tmule config

File: rasberry_bringup/urdf/robot_014_sensors_corner_hokuyos.xacro (robot description, xacro)
@@ -53,12 +53,12 @@
   </joint>
   <joint name="base_sens_septentrio" type="fixed">
-    <parent link="$(arg tf_prefix)/base_sensors"/>
+    <parent link="$(arg tf_prefix)/base_link"/>
     <child link="$(arg tf_prefix)/septentrio"/>
-    <origin xyz="-0.01 0 0.3" rpy="0 0 0"/>
+    <origin xyz="-0.5325 -0.314 0.814" rpy="0 0 0"/>
   </joint>
   <joint name="base_sens_xsens" type="fixed">
     <parent link="$(arg tf_prefix)/base_link"/>
     <child link="$(arg tf_prefix)/xsens"/>
-    <origin xyz="-0.005 0.2605 0.682" rpy="0 0 0"/>
+    <origin xyz="0.18 -0.266 0.717" rpy="0 0 0"/>
   </joint>
    <joint name="base_sens_hokuyo_front" type="fixed">

Commit message: Updated xacro files for Ouster on 014 and 019

File: rasberry_bringup/urdf/robot_014_sensors_corner_hokuyos.xacro (robot description, xacro)
@@ -6,5 +6,5 @@
   <link name="$(arg tf_prefix)/septentrio"/>
   <link name="$(arg tf_prefix)/xsens"/>
-  <link name="$(arg tf_prefix)/velodyne"/>
+  <link name="$(arg tf_prefix)/os1_sensor"/>
   <!-- Hokuyo Laser -->
   <link name="$(arg tf_prefix)/hokuyo_front">
@@ -74,7 +74,7 @@
     <origin xyz="0.172 -0.152 -0.034" rpy="0.0 0.0 -0.79"/>
   </joint>
- <joint name="base_sens_velodyne" type="fixed">
+ <joint name="base_sens_ouster" type="fixed">
     <parent link="$(arg tf_prefix)/base_sensors"/>
-    <child link="$(arg tf_prefix)/velodyne"/>
+    <child link="$(arg tf_prefix)/os1_sensor"/>
     <axis xyz="0 1 0" />
     <origin xyz="0 0 0" rpy="0 0 0"/>

File: rasberry_bringup/urdf/robot_019_sensors_corner_hokuyos.xacro (robot description, xacro)
@@ -6,5 +6,5 @@
   <link name="$(arg tf_prefix)/septentrio"/>
   <link name="$(arg tf_prefix)/xsens"/>
-  <link name="$(arg tf_prefix)/velodyne"/>
+  <link name="$(arg tf_prefix)/os1_sensor"/>
   <!-- Hokuyo Laser -->
   <link name="$(arg tf_prefix)/hokuyo_front">
@@ -74,9 +74,9 @@
     <origin xyz="0.172 -0.152 -0.034" rpy="0.0 0.0 -0.79"/>
   </joint>
- <joint name="base_sens_velodyne" type="fixed">
+ <joint name="base_sens_ouster" type="fixed">
     <parent link="$(arg tf_prefix)/base_sensors"/>
-    <child link="$(arg tf_prefix)/velodyne"/>
+    <child link="$(arg tf_prefix)/os1_sensor"/>
     <axis xyz="0 1 0" />
-    <origin xyz="0 0 0" rpy="0 0 3.14159"/>
+    <origin xyz="0 0 0" rpy="0 0 0"/>
   </joint>
   <!--hokuyo-->

Commit message: ekf local localisation using imu

File: rasberry_bringup/urdf/robot_014_sensors_corner_hokuyos.xacro (robot description, xacro)
@@ -61,4 +61,9 @@
     <child link="$(arg tf_prefix)/xsens"/>
     <origin xyz="0.18 -0.266 0.717" rpy="0 0 0"/>
+  </joint>
+  <joint name="base_sens_um7" type="fixed">
+    <parent link="$(arg tf_prefix)/base_link"/>
+    <child link="$(arg tf_prefix)/imu_link"/>
+    <origin xyz="0.20 0.16 0.69" rpy="0 0 0"/>
   </joint>
    <joint name="base_sens_hokuyo_front" type="fixed">

File: rasberry_bringup/urdf/robot_019_sensors_corner_hokuyos.xacro (robot description, xacro)
@@ -61,4 +61,9 @@
     <child link="$(arg tf_prefix)/xsens"/>
     <origin xyz="0.18 -0.266 0.717" rpy="0 0 0"/>
+  </joint>
+  <joint name="base_sens_um7" type="fixed">
+    <parent link="$(arg tf_prefix)/base_link"/>
+    <child link="$(arg tf_prefix)/imu_link"/>
+    <origin xyz="0.20 0.16 0.69" rpy="0 0 0"/>
   </joint>
    <joint name="base_sens_hokuyo_front" type="fixed">

Commit message: missed link name for imu_link

File: rasberry_bringup/urdf/robot_014_sensors_corner_hokuyos.xacro (robot description, xacro)
@@ -7,4 +7,5 @@
   <link name="$(arg tf_prefix)/xsens"/>
   <link name="$(arg tf_prefix)/os1_sensor"/>
+  <link name="$(arg tf_prefix)/imu_link"/>
   <!-- Hokuyo Laser -->
   <link name="$(arg tf_prefix)/hokuyo_front">

File: rasberry_bringup/urdf/robot_019_sensors_corner_hokuyos.xacro (robot description, xacro)
@@ -7,4 +7,5 @@
   <link name="$(arg tf_prefix)/xsens"/>
   <link name="$(arg tf_prefix)/os1_sensor"/>
+  <link name="$(arg tf_prefix)/imu_link"/>
   <!-- Hokuyo Laser -->
   <link name="$(arg tf_prefix)/hokuyo_front">
